File: kicad/subsheets/rv1106.kicad_sch (KiCad schematic)
At the start: 58 parts, among them U4 RV1106G2

Commit message: Add missing passives and microphone
Parts:
- removed R21: 100R, Resistor_SMD:R_0402_1005Metric, symbol Device:R_Small
- added C59, C73, C74, C81: 100nF, Capacitor_SMD:C_0402_1005Metric, symbol Device:C_Small
- added C80, C85: 1uF, Capacitor_SMD:C_0603_1608Metric, symbol Device:C_Small
- added C82, C83, C84: 100pF, Capacitor_SMD:C_0402_1005Metric, symbol Device:C_Small
- added MIC1: IM73A135V01, Sensor_Audio:Infineon_PG-LLGA-5-2, symbol Sensor_Audio:IM73A135V01
- added R19, R22, R32, R33: 10k, Resistor_SMD:R_0603_1608Metric, symbol Device:R_Small
- added R39, R40: 22k, Resistor_SMD:R_0402_1005Metric, symbol Device:R_Small
- renumbered C42 to C41, C43 to C42, C44 to C43, C45 to C44, C46 to C45, C47 to C46, C48 to C47, C49 to C48, C50 to C49, C51 to C50, C52 to C51, C53 to C52, C54 to C53, C55 to C54, C56 to C55, C57 to C56, C58 to C57, C59 to C58, C64 to C63, C63 to C64, C71 to C66, C72 to C67, C67 to C69, C73 to C70, C74 to C71, C70 to C72, C66 to C75, C69 to C76, C75 to C77, C76 to C78, C77 to C79, R19 to R20, R20 to R21, R22 to R23, R23 to R24, R33 to R25, R34 to R26, R24 to R27, R27 to R28, R28 to R29, R25 to R30, R26 to R31, R32 to R34, R29 to R35, R30 to R36, R31 to R37
Connections:
- net GND: now also C59.2, C73.2, C74.2, C81.2, C83.1, C84.2, MIC1.4 (GND), MIC1.5 (GND), R22.2
- net VCC_1V8: now also R32.1, R33.2
- net at U4.22 (SARADC_IN1/PWM1_M1/GPI4_C1_z): now also C73.1, R32.2
- net RECOVER: now reaches U4.23 (SARADC_IN0/GPI4_C0_z)
- net RECOVER: now also C74.1, R33.1
- net USB_VBUSDET: now reaches U4.25 (USB_VBUSDET)
- net USB_VBUSDET: now also C59.1, R19.2, R22.1
- net VCC1V8_MICBIAS: now reaches U4.32 (CODEC_MICBIAS)
- net VCC1V8_MICBIAS: now also C81.1, MIC1.2 (V_{DD})
- net at U4.33 (CODEC_MIC0N): now also C80.1
- net at U4.34 (CODEC_MIC0P): now also C85.1
- new net: C82.2, C84.1, MIC1.3 (OUT-), R40.2
- new net: C82.1, C83.2, MIC1.1 (OUT+), R39.2
- new net CODEC_MIC0N: C80.2, R40.1
- new net CODEC_MIC0P: C85.2, R39.1
- new net USB_VBUS_5V: R19.1
- no-connect marks 55 -> 57
Other:
- note removed: "!"
- moved on the sheet: C41, C42, C43, C44, C45, C46, C47, C48, C49, C50, C51, C52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
