File: kicad/subsheets/rv1106.kicad_sch (KiCad schematic)
At the start: 73 parts, among them U4 RV1106G2

Commit message: Footprint + silkscreen corrections
Parts:
- C41: renamed from C60; now left out of the parts list
- C42: renamed from C41; now left out of the parts list
- C43: renamed from C61; now left out of the parts list
- C44: renamed from C62; now left out of the parts list
- C45: renamed from C51; now left out of the parts list
- C46: renamed from C80; now left out of the parts list
- C47: renamed from C85; now left out of the parts list
- C48: renamed from C72; now left out of the parts list
- C49: renamed from C76; now left out of the parts list
- C50: renamed from C75; now left out of the parts list
- C51: renamed from C73; now left out of the parts list
- C52: renamed from C68; now left out of the parts list
- C53: renamed from C69; now left out of the parts list
- C54: renamed from C74; now left out of the parts list
- C55: renamed from C63; now left out of the parts list
- C56: renamed from C64; now left out of the parts list
- C57: renamed from C65; now left out of the parts list
- C58: renamed from C79; now left out of the parts list
- C59: renamed from C77; now left out of the parts list
- C60: renamed from C78; now left out of the parts list
- C61: renamed from C42; now left out of the parts list
- C62: renamed from C43; now left out of the parts list
- C63: renamed from C59; now left out of the parts list
- C64: renamed from C44; now left out of the parts list
- C65: renamed from C70; now left out of the parts list
- C66: renamed from C71; now left out of the parts list
- C67: renamed from C66; now left out of the parts list
- C68: renamed from C83; now left out of the parts list
- C69: renamed from C82; now left out of the parts list
- C70: renamed from C84; now left out of the parts list
- C71: renamed from C45; now left out of the parts list
- C72: renamed from C67; now left out of the parts list
- C73: renamed from C52; now left out of the parts list
- C74: renamed from C46; now left out of the parts list
- C75: renamed from C53; now left out of the parts list
- C76: renamed from C47; now left out of the parts list
- C77: renamed from C81; now left out of the parts list
- C78: renamed from C54; now left out of the parts list
- C79: renamed from C55; now left out of the parts list
- C80: renamed from C48; now left out of the parts list
- C81: renamed from C56; now left out of the parts list
- C82: renamed from C49; now left out of the parts list
- C83: renamed from C57; now left out of the parts list
- C84: renamed from C50; now left out of the parts list
- C85: renamed from C58; now left out of the parts list
- FB4, MIC1: now left out of the parts list
- HSE1: renamed from HSE2; now left out of the parts list
- HSE2: renamed from HSE1; now left out of the parts list
- R18: renamed from R20; now left out of the parts list
- R19: renamed from R21; now left out of the parts list
- R21: renamed from R18; now left out of the parts list
- R22: renamed from R23; now left out of the parts list
- R23: renamed from R27; now left out of the parts list
- R24: renamed from R34; now left out of the parts list
- R25: renamed from R30; now left out of the parts list
- R26: renamed from R31; now left out of the parts list
- R27: renamed from R32; now left out of the parts list
- R28: renamed from R33; now left out of the parts list
- R29: renamed from R37; now left out of the parts list
- R30: renamed from R35; now left out of the parts list
- R31: renamed from R36; now left out of the parts list
- R32: renamed from R19; now left out of the parts list
- R33: renamed from R22; now left out of the parts list
- R34: renamed from R39; now left out of the parts list
- R35: renamed from R40; now left out of the parts list
- R36: renamed from R28; now left out of the parts list
- R38: renamed from R29; now left out of the parts list
- renumbered R24 to R20, R25 to R37, R26 to R39

Commit message: Final changes before order
Parts:
- removed C68, C69, C70: 100pF, Capacitor_SMD:C_0402_1005Metric, symbol Device:C_Small
- removed C77: 100nF, Capacitor_SMD:C_0402_1005Metric, symbol Device:C_Small
- removed MIC1: IM73A135V01, Sensor_Audio:Infineon_PG-LLGA-5-2, symbol Sensor_Audio:IM73A135V01
- removed R34, R35: 22k, Resistor_SMD:R_0402_1005Metric, symbol Device:R_Small
- added C86: 100nF, Capacitor_SMD:C_0402_1005Metric, symbol Device:C_Small
- added C87: 15pF, Capacitor_SMD:C_0402_1005Metric, symbol Device:C_Small
- added FB5: 120R, Resistor_SMD:R_0603_1608Metric, symbol Device:FerriteBead_Small
- added MIC1: CMM-2718AB-3815NC-TR, a3-srad-camera-v2:MIC_CMM-2718AB-3815NC-TR, symbol a3-srad-camera-v2:CMM-2718AB-3815NC-TR
- added NT1: NetTie_2, symbol Device:NetTie_2
- C46, C47: value 1uF -> 100nF; footprint Capacitor_SMD:C_0603_1608Metric -> Capacitor_SMD:C_0402_1005Metric
Connections:
- net CODEC_MIC0N: now also NT1.2
- net CODEC_MIC0P: now also C87.1, MIC1.2 (OUTPUT)
- net GND: now also C86.2, C87.2, MIC1.3 (GND), NT1.1
- net VCC1V8_MICBIAS: now also FB5.1
- new net: C86.1, FB5.2, MIC1.1 (VDD)

Commit message: Minor kicad changes
Parts:
- C41, C42, C43, C45, C46, C47, C49, C50, C53, C55, C56, C59, C63, C65, C66, C67, C71, C72, C75, C78, C81, C82, C83, C84, C85, FB4, FB5, HSE1, HSE2, R18, R19: BOARD_SIDE (none) -> Front; now in the parts list
- C44, C48, C51, C52, C54, C57, C58, C60, C61, C62, C64, C73, C74, C76, C79, C80, C86, C87, JP2, NT1, R20, R21, R22, R23, R24, R25, R26, R27, R28, R29, R30, R31, R32, R33, R36, R37, R38, R39: now in the parts list
- MIC1, U4: BOARD_SIDE (none) -> Front
